File: matrix-mixer/matrix-mixer.sch (KiCad schematic (older format))
At the start: 46 parts, among them J5 JACK-MONO, J6 JACK-MONO, J7 JACK-MONO, J8 JACK-MONO, J9 EURO_HEADER_10pin, SW5 SW_SPDT, SW6 SW_SPDT, SW7 SW_SPDT, SW8 SW_SPDT, U1 LM324

Commit message: matrix 0.0.1
Parts:
- removed C1, C2, C3, C4: C, symbol 4ms-passives:C
- removed J6, J7, J8: JACK-MONO, symbol 4ms-mech:JACK-MONO
- removed RV2, RV3, RV4: R_POT, symbol Device:R_POT
- removed SW5, SW6, SW7, SW8: SW_SPDT, symbol 4ms-mech:SW_SPDT
- removed U1: LM324, symbol 4ms-ic:LM324
- added IC1: LM324N, 4ms_Package_DIP:DIP-14_W7.62mm, symbol matrix-mixer-eagle-import:LM324N
- added J3, J4, J5: JACK-MONO, Eurocad:PJ301M-12, symbol 4ms-mech:JACK-MONO
- added R10, R11, R12, R13, R14, R15, R16, R5, R6, R7, R8, R9: 100k, Resistor_THT:R_Axial_DIN0207_L6.3mm_D2.5mm_P7.62mm_Horizontal, symbol 4ms-passives:R
- added RV13, RV5, RV9: R_POT, 4ms-footprints:POT-9MM-ALPHA, symbol Device:R_POT
- INPUT_A1: renamed from INPUT_A; footprint (none) -> Eurocad:PJ301M-12
- INPUT_B1: renamed from INPUT_B; footprint (none) -> Eurocad:PJ301M-12
- INPUT_C1: renamed from INPUT_C; footprint (none) -> Eurocad:PJ301M-12
- INPUT_D1: renamed from INPUT_D; footprint (none) -> Eurocad:PJ301M-12
- J2: renamed from J5; footprint (none) -> Eurocad:PJ301M-12
- MUTE_A1: renamed from MUTE_A; footprint (none) -> 4ms-footprints:SPST-SUB
- MUTE_B1: renamed from MUTE_B; footprint (none) -> 4ms-footprints:SPST-SUB
- MUTE_C1: renamed from MUTE_C; footprint (none) -> 4ms-footprints:SPST-SUB
- MUTE_D1: renamed from MUTE_D; footprint (none) -> 4ms-footprints:SPST-SUB
- R1, R2, R3, R4: value R -> 100k; footprint (none) -> Resistor_THT:R_Axial_DIN0207_L6.3mm_D2.5mm_P7.62mm_Horizontal
- RV1, RV10, RV11, RV12, RV14, RV15, RV16, RV6, RV7, RV8: footprint (none) -> 4ms-footprints:POT-9MM-ALPHA
- RV2: renamed from RV5; footprint (none) -> 4ms-footprints:POT-9MM-ALPHA
- RV3: renamed from RV9; footprint (none) -> 4ms-footprints:POT-9MM-ALPHA
- RV4: renamed from RV13; footprint (none) -> 4ms-footprints:POT-9MM-ALPHA
- gave numbers to parts that had none: 4
- renumbered J9 to J1
Connections:
- wire segments 31 -> 194
- no-connect marks 0 -> 8
Other:
- moved on the sheet: C1, C2, D1, D2, INPUT_A1, INPUT_B1, INPUT_C1, INPUT_D1, J1, J2, MUTE_A1, MUTE_B1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

Commit message: matrix 0.0.2 but not routed
Parts:
- removed MUTE_A1, MUTE_B1, MUTE_C1, MUTE_D1: SW_SPST, 4ms-footprints:SPST-SUB, symbol Switch:SW_SPST
- added IC2: LM324N, 4ms_Package_DIP:DIP-14_W7.62mm, symbol matrix-mixer-eagle-import:LM324N
- added R17, R20, R23, R26: 70k, 4ms_Resistor:R_Axial_DIN0207_L6.3mm_D2.5mm_P7.62mm_Horizontal, symbol 4ms-passives:R
- added R18, R19, R21, R22, R24, R25, R27, R28: 100k, 4ms_Resistor:R_Axial_DIN0207_L6.3mm_D2.5mm_P7.62mm_Horizontal, symbol 4ms-passives:R
- renumbered J2 to OUTPUT_A1, J3 to OUTPUT_B1, J4 to OUTPUT_C1, J5 to OUTPUT_D1
Connections:
- wire segments 194 -> 252
- no-connect marks 8 -> 7
Other:
- moved on the sheet: OUTPUT_A1, OUTPUT_B1, OUTPUT_C1, OUTPUT_D1, R1, R10, R11, R12, R13, R14, R15, R16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

Commit message: matrix mixer 0.0.2 routed ready to send
Parts:
- removed INPUT_A1, OUTPUT_A1, OUTPUT_B1, OUTPUT_C1, OUTPUT_D1: JACK-MONO, Eurocad:PJ301M-12, symbol 4ms-mech:JACK-MONO
- removed INPUT_B1, INPUT_C1, INPUT_D1: JACK_MONO, Eurocad:PJ301M-12, symbol 4ms-mech:JACK-MONO
- added INPUT_A1, INPUT_B1, INPUT_C1, INPUT_D1, OUTPUT_A1, OUTPUT_B1, OUTPUT_C1, OUTPUT_D1: THONKICONNNEW, Connector_Audio:Jack_3.5mm_QingPu_WQP-PJ398SM_Vertical_CircularHoles, symbol matrix-mixer-eagle-import:THONKICONNNEW
Connections:
- net GND: now also IC1.3 (+IN), IC1.5 (+IN), IC2.3 (+IN), IC2.5 (+IN), INPUT_A1.P$3_GND (GND), INPUT_B1.P$3_GND (GND), INPUT_C1.P$3_GND (GND), INPUT_D1.P$3_GND (GND), OUTPUT_A1.P$3_GND (GND), OUTPUT_B1.P$3_GND (GND), OUTPUT_C1.P$3_GND (GND), OUTPUT_D1.P$3_GND (GND); no longer IC1.3 (+IN), IC1.5 (+IN), IC2.3 (+IN), IC2.5 (+IN)
- net at RV1.3, RV2.3, RV3.3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: now also INPUT_A1.P$1_TIP (T)
- net at RV5.3, RV6.3, RV7.3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: now also INPUT_B1.P$1_TIP (T)
- net at RV10.3, RV11.3, RV12.3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: now also INPUT_C1.P$1_TIP (T)
- net at RV13.3, RV14.3, RV15.3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: now also INPUT_D1.P$1_TIP (T)
- net at R19.2: now also IC1.1 (OUT), OUTPUT_A1.P$1_TIP (T); no longer IC1.7 (OUT)
- net at D1.2 (A), J1.1 (+12V): now also J1.2 (+12V)
- net at J1.10 (-12V): now also D2.1 (K), J1.9 (-12V)
- net at R1.2, R13.2, R17.1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: now also IC1.6 (-IN); no longer IC1.2 (-IN)
- net at R11.2, R15.2, R23.1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: now also IC2.6 (-IN); no longer IC2.2 (-IN)
- net at IC1.14 (OUT), R22.2: now also OUTPUT_B1.P$1_TIP (T)
- net at R25.2: now also IC2.1 (OUT), OUTPUT_C1.P$1_TIP (T); no longer IC2.7 (OUT)
- net at IC2.14 (OUT), R28.2: now also OUTPUT_D1.P$1_TIP (T)
- net at R18.2, R19.1: now also IC1.2 (-IN); no longer IC1.6 (-IN)
- net at R17.2, R18.1: now also IC1.7 (OUT); no longer IC1.1 (OUT)
- net at R24.2, R25.1: now also IC2.2 (-IN); no longer IC2.6 (-IN)
- net at R23.2, R24.1: now also IC2.7 (OUT); no longer IC2.1 (OUT)
- no-connect marks 7 -> 3
